File: Control.sch (EAGLE design)
At the start: 44 parts, among them IC2 7805T, IC3 LP2950Z, Q2 16MHZ, X1 BUT4, X10 DIG2, X11 DIG3, X12 DIG4, X2 BUT3, X3 AL1, X4 BUT2, X5 BUT1, X6 AL2, X7 AL3, X8 AL4, X9 DIG1

Commit message: 28/10/13
Fixed:
-Relay PCB
-half Control PCB

unfixed:
-Control PCB GND separation
Parts:
- renumbered PDM to PDBUT2, PDM1 to PDBUT4, PDS to PDBUT1, PDS1 to PDBUT3
Changed lines of the file:
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@@
 <part name="X5" library="con-molex" deviceset="22-23-2021" device="" value="BUT1"/>
 <part name="P+6" library="supply1" deviceset="+5V" device=""/>
-<part name="PDM" library="adafruit" deviceset="R-US_" device="0204/7" value="10k"/>
-<part name="PDS" library="adafruit" deviceset="R-US_" device="0204/7" value="10k"/>
+<part name="PDBUT2" library="adafruit" deviceset="R-US_" device="0204/7" value="10k"/>
+<part name="PDBUT1" library="adafruit" deviceset="R-US_" device="0204/7" value="10k"/>
 <part name="SUPPLY16" library="supply2" deviceset="GND" device=""/>
 <part name="SUPPLY17" library="supply2" deviceset="GND" device=""/>
@@
 <part name="X2" library="con-molex" deviceset="22-23-2021" device="" value="BUT3"/>
 <part name="P+8" library="supply1" deviceset="+5V" device=""/>
-<part name="PDM1" library="adafruit" deviceset="R-US_" device="0204/7" value="10k"/>
-<part name="PDS1" library="adafruit" deviceset="R-US_" device="0204/7" value="10k"/>
+<part name="PDBUT4" library="adafruit" deviceset="R-US_" device="0204/7" value="10k"/>
+<part name="PDBUT3" library="adafruit" deviceset="R-US_" device="0204/7" value="10k"/>
 <part name="SUPPLY2" library="supply2" deviceset="GND" device=""/>
 <part name="SUPPLY3" library="supply2" deviceset="GND" device=""/>
@@
 <instance part="X5" gate="-2" x="-198.12" y="68.58" rot="R180"/>
 <instance part="P+6" gate="1" x="-195.58" y="76.2"/>
-<instance part="PDM" gate="G$1" x="-170.18" y="53.34" rot="R90"/>
-<instance part="PDS" gate="G$1" x="-195.58" y="53.34" rot="R90"/>
+<instance part="PDBUT2" gate="G$1" x="-170.18" y="53.34" rot="R90"/>
+<instance part="PDBUT1" gate="G$1" x="-195.58" y="53.34" rot="R90"/>
 <instance part="SUPPLY16" gate="GND" x="-170.18" y="43.18"/>
 <instance part="SUPPLY17" gate="GND" x="-195.58" y="43.18"/>
@@
 <instance part="X2" gate="-2" x="-144.78" y="68.58" rot="R180"/>
 <instance part="P+8" gate="1" x="-142.24" y="76.2"/>
-<instance part="PDM1" gate="G$1" x="-116.84" y="53.34" rot="R90"/>
-<instance part="PDS1" gate="G$1" x="-142.24" y="53.34" rot="R90"/>
+<instance part="PDBUT4" gate="G$1" x="-116.84" y="53.34" rot="R90"/>
+<instance part="PDBUT3" gate="G$1" x="-142.24" y="53.34" rot="R90"/>
 <instance part="SUPPLY2" gate="GND" x="-116.84" y="43.18"/>
 <instance part="SUPPLY3" gate="GND" x="-142.24" y="43.18"/>
@@
 </segment>
 <segment>
-<pinref part="PDM" gate="G$1" pin="1"/>
+<pinref part="PDBUT2" gate="G$1" pin="1"/>
 <wire x1="-170.18" y1="48.26" x2="-170.18" y2="45.72" width="0.1524" layer="91"/>
 <pinref part="SUPPLY16" gate="GND" pin="GND"/>
 </segment>
 <segment>
-<pinref part="PDS" gate="G$1" pin="1"/>
+<pinref part="PDBUT1" gate="G$1" pin="1"/>
 <wire x1="-195.58" y1="48.26" x2="-195.58" y2="45.72" width="0.1524" layer="91"/>
 <pinref part="SUPPLY17" gate="GND" pin="GND"/>
@@
 </segment>
 <segment>
-<pinref part="PDM1" gate="G$1" pin="1"/>
+<pinref part="PDBUT4" gate="G$1" pin="1"/>
 <wire x1="-116.84" y1="48.26" x2="-116.84" y2="45.72" width="0.1524" layer="91"/>
 <pinref part="SUPPLY2" gate="GND" pin="GND"/>
 </segment>
 <segment>
-<pinref part="PDS1" gate="G$1" pin="1"/>
+<pinref part="PDBUT3" gate="G$1" pin="1"/>
 <wire x1="-142.24" y1="48.26" x2="-142.24" y2="45.72" width="0.1524" layer="91"/>
 <pinref part="SUPPLY3" gate="GND" pin="GND"/>
@@
 <wire x1="-116.84" y1="60.96" x2="-109.22" y2="60.96" width="0.1524" layer="91"/>
 <junction x="-116.84" y="60.96"/>
-<pinref part="PDM1" gate="G$1" pin="2"/>
+<pinref part="PDBUT4" gate="G$1" pin="2"/>
 <label x="-109.22" y="60.96" size="1.778" layer="95"/>
 </segment>
@@
 <wire x1="-170.18" y1="60.96" x2="-162.56" y2="60.96" width="0.1524" layer="91"/>
 <junction x="-170.18" y="60.96"/>
-<pinref part="PDM" gate="G$1" pin="2"/>
+<pinref part="PDBUT2" gate="G$1" pin="2"/>
 <label x="-162.56" y="60.96" size="1.778" layer="95"/>
 </segment>
@@
 <wire x1="-142.24" y1="60.96" x2="-134.62" y2="60.96" width="0.1524" layer="91"/>
 <junction x="-142.24" y="60.96"/>
-<pinref part="PDS1" gate="G$1" pin="2"/>
+<pinref part="PDBUT3" gate="G$1" pin="2"/>
 <label x="-134.62" y="60.96" size="1.778" layer="95"/>
 </segment>
@@
 <wire x1="-195.58" y1="60.96" x2="-187.96" y2="60.96" width="0.1524" layer="91"/>
 <junction x="-195.58" y="60.96"/>
-<pinref part="PDS" gate="G$1" pin="2"/>
+<pinref part="PDBUT1" gate="G$1" pin="2"/>
 <label x="-187.96" y="60.96" size="1.778" layer="95"/>
 </segment>

Commit message: 28/10/13 - 2
Fixed:
-Relay & Control PCB

Unfixed:
-IR PCB
-Temperature PCB
Connections:
- net +5V: now also JP2.1
- net VCC: no longer JP2.1
Changed lines of the file:
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@@
 <part name="XON" library="adafruit" deviceset="LED" device="3MM"/>
 <part name="P+18" library="supply1" deviceset="+5V" device=""/>
-<part name="GND1" library="SparkFun-Aesthetics" deviceset="GND" device="" value="AGND"/>
-<part name="GND4" library="SparkFun-Aesthetics" deviceset="GND" device="" value="AGND"/>
 <part name="SUPPLY1" library="supply2" deviceset="GND" device=""/>
-<part name="GND2" library="SparkFun-Aesthetics" deviceset="GND" device="" value="AGND"/>
 <part name="AGND" library="adafruit" deviceset="PINHD-1X1" device="" value="AGND"/>
-<part name="GND5" library="SparkFun-Aesthetics" deviceset="GND" device="" value="AGND"/>
 <part name="X1" library="con-molex" deviceset="22-23-2021" device="" value="BUT4"/>
 <part name="P+7" library="supply1" deviceset="+5V" device=""/>
@@
 <part name="X6" library="con-molex" deviceset="22-23-2031" device="" value="AL2"/>
 <part name="P+9" library="supply1" deviceset="+5V" device=""/>
-<part name="GND3" library="SparkFun-Aesthetics" deviceset="GND" device="" value="AGND"/>
 <part name="X7" library="con-molex" deviceset="22-23-2031" device="" value="AL3"/>
 <part name="P+10" library="supply1" deviceset="+5V" device=""/>
-<part name="GND6" library="SparkFun-Aesthetics" deviceset="GND" device="" value="AGND"/>
 <part name="X8" library="con-molex" deviceset="22-23-2031" device="" value="AL4"/>
 <part name="P+11" library="supply1" deviceset="+5V" device=""/>
-<part name="GND7" library="SparkFun-Aesthetics" deviceset="GND" device="" value="AGND"/>
 <part name="X9" library="con-molex" deviceset="22-23-2031" device="" value="DIG1"/>
 <part name="P+12" library="supply1" deviceset="+5V" device=""/>
@@
 <part name="PSCL" library="adafruit" deviceset="R-US_" device="0204/7" value="4k7"/>
 <part name="P+19" library="supply1" deviceset="+5V" device=""/>
+<part name="AGND1" library="supply1" deviceset="AGND" device=""/>
+<part name="AGND2" library="supply1" deviceset="AGND" device=""/>
+<part name="AGND3" library="supply1" deviceset="AGND" device=""/>
+<part name="AGND4" library="supply1" deviceset="AGND" device=""/>
+<part name="AGND5" library="supply1" deviceset="AGND" device=""/>
+<part name="AGND6" library="supply1" deviceset="AGND" device=""/>
+<part name="AGND7" library="supply1" deviceset="AGND" device=""/>
 </parts>
 <sheets>
@@
 <instance part="XON" gate="G$1" x="-38.1" y="127"/>
 <instance part="P+18" gate="1" x="-175.26" y="149.86"/>
-<instance part="GND1" gate="1" x="-68.58" y="71.12"/>
-<instance part="GND4" gate="1" x="30.48" y="104.14"/>
 <instance part="SUPPLY1" gate="GND" x="38.1" y="99.06"/>
-<instance part="GND2" gate="1" x="25.4" y="111.76"/>
 <instance part="AGND" gate="G$1" x="-205.74" y="129.54" rot="R180"/>
-<instance part="GND5" gate="1" x="-195.58" y="124.46"/>
 <instance part="X1" gate="-1" x="-119.38" y="66.04" rot="R180"/>
 <instance part="X1" gate="-2" x="-119.38" y="68.58" rot="R180"/>
@@
 <instance part="X6" gate="-3" x="-50.8" y="83.82" rot="R180"/>
 <instance part="P+9" gate="1" x="-43.18" y="91.44"/>
-<instance part="GND3" gate="1" x="-43.18" y="71.12"/>
 <instance part="X7" gate="-1" x="-22.86" y="78.74" rot="R180"/>
 <instance part="X7" gate="-2" x="-22.86" y="81.28" rot="R180"/>
 <instance part="X7" gate="-3" x="-22.86" y="83.82" rot="R180"/>
 <instance part="P+10" gate="1" x="-15.24" y="91.44"/>
-<instance part="GND6" gate="1" x="-15.24" y="71.12"/>
 <instance part="X8" gate="-1" x="2.54" y="78.74" rot="R180"/>
 <instance part="X8" gate="-2" x="2.54" y="81.28" rot="R180"/>
 <instance part="X8" gate="-3" x="2.54" y="83.82" rot="R180"/>
 <instance part="P+11" gate="1" x="10.16" y="91.44"/>
-<instance part="GND7" gate="1" x="10.16" y="71.12"/>
 <instance part="X9" gate="-1" x="-76.2" y="48.26" rot="R180"/>
 <instance part="X9" gate="-2" x="-76.2" y="50.8" rot="R180"/>
@@
 <instance part="PSCL" gate="G$1" x="78.74" y="53.34" rot="R90"/>
 <instance part="P+19" gate="1" x="83.82" y="66.04"/>
+<instance part="AGND1" gate="VR1" x="-195.58" y="124.46"/>
+<instance part="AGND2" gate="VR1" x="-68.58" y="71.12"/>
+<instance part="AGND3" gate="VR1" x="-43.18" y="71.12"/>
+<instance part="AGND4" gate="VR1" x="-15.24" y="71.12"/>
+<instance part="AGND5" gate="VR1" x="10.16" y="71.12"/>
+<instance part="AGND6" gate="VR1" x="30.48" y="104.14"/>
+<instance part="AGND7" gate="VR1" x="25.4" y="111.76"/>
 </instances>
 <busses>
@@
 <wire x1="55.88" y1="76.2" x2="45.72" y2="76.2" width="0.1524" layer="91"/>
 <label x="45.72" y="76.2" size="1.778" layer="95"/>
-</segment>
-<segment>
-<pinref part="JP2" gate="A" pin="1"/>
-<wire x1="55.88" y1="45.72" x2="45.72" y2="45.72" width="0.1524" layer="91"/>
-<label x="45.72" y="45.72" size="1.778" layer="95"/>
 </segment>
 </net>
@@
 <pinref part="P+19" gate="1" pin="+5V"/>
 </segment>
+<segment>
+<pinref part="JP2" gate="A" pin="1"/>
+<wire x1="55.88" y1="45.72" x2="45.72" y2="45.72" width="0.1524" layer="91"/>
+<label x="45.72" y="45.72" size="1.778" layer="95"/>
+</segment>
 </net>
 <net name="DIG3" class="0">
@@
 <wire x1="40.64" y1="119.38" x2="30.48" y2="119.38" width="0.1524" layer="91"/>
 <wire x1="30.48" y1="119.38" x2="30.48" y2="106.68" width="0.1524" layer="91"/>
-<pinref part="GND4" gate="1" pin="GND"/>
+<pinref part="AGND6" gate="VR1" pin="AGND"/>
 </segment>
 <segment>
@@
 <wire x1="-73.66" y1="78.74" x2="-68.58" y2="78.74" width="0.1524" layer="91"/>
 <wire x1="-68.58" y1="78.74" x2="-68.58" y2="73.66" width="0.1524" layer="91"/>
-<pinref part="GND1" gate="1" pin="GND"/>
+<pinref part="AGND2" gate="VR1" pin="AGND"/>
 </segment>
 <segment>
 <wire x1="25.4" y1="116.84" x2="25.4" y2="114.3" width="0.1524" layer="91"/>
 <pinref part="REF" gate="G$1" pin="2"/>
-<pinref part="GND2" gate="1" pin="GND"/>
+<pinref part="AGND7" gate="VR1" pin="AGND"/>
 </segment>
 <segment>
@@
 <wire x1="-203.2" y1="129.54" x2="-195.58" y2="129.54" width="0.1524" layer="91"/>
 <wire x1="-195.58" y1="129.54" x2="-195.58" y2="127" width="0.1524" layer="91"/>
-<pinref part="GND5" gate="1" pin="GND"/>
+<pinref part="AGND1" gate="VR1" pin="AGND"/>
 </segment>
 <segment>
@@
 <wire x1="-48.26" y1="78.74" x2="-43.18" y2="78.74" width="0.1524" layer="91"/>
 <wire x1="-43.18" y1="78.74" x2="-43.18" y2="73.66" width="0.1524" layer="91"/>
-<pinref part="GND3" gate="1" pin="GND"/>
+<pinref part="AGND3" gate="VR1" pin="AGND"/>
 </segment>
 <segment>
@@
 <wire x1="-20.32" y1="78.74" x2="-15.24" y2="78.74" width="0.1524" layer="91"/>
 <wire x1="-15.24" y1="78.74" x2="-15.24" y2="73.66" width="0.1524" layer="91"/>
-<pinref part="GND6" gate="1" pin="GND"/>
+<pinref part="AGND4" gate="VR1" pin="AGND"/>
 </segment>
 <segment>
@@
 <wire x1="5.08" y1="78.74" x2="10.16" y2="78.74" width="0.1524" layer="91"/>
 <wire x1="10.16" y1="78.74" x2="10.16" y2="73.66" width="0.1524" layer="91"/>
-<pinref part="GND7" gate="1" pin="GND"/>
-</segment>
-</net>
+<pinref part="AGND5" gate="VR1" pin="AGND"/>
+</segment>
+</net>
