File: Control.sch (EAGLE design)
At the start: 44 parts, among them IC2 7805T, IC3 LP2950Z, Q2 16MHZ, X1 BUT4, X10 DIG2, X11 DIG3, X12 DIG4, X2 BUT3, X3 AL1, X4 BUT2, X5 BUT1, X6 AL2, X7 AL3, X8 AL4, X9 DIG1

Commit message: 13/11/13
Fixed:
-Resistor Value
Parts:
- RXASC, RXON: value 220 -> 10K
Changed lines of the file:
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@@
 <part name="SUPPLY31" library="supply2" deviceset="GND" device=""/>
 <part name="SUPPLY32" library="supply2" deviceset="GND" device=""/>
-<part name="RXASC" library="adafruit" deviceset="R-US_" device="0204/7" value="220"/>
+<part name="RXASC" library="adafruit" deviceset="R-US_" device="0204/7" value="10K"/>
 <part name="XASC" library="adafruit" deviceset="LED" device="3MM"/>
 <part name="RSSI1" library="adafruit" deviceset="PINHD-1X1" device=""/>
@@
 <part name="SUPPLY13" library="supply2" deviceset="GND" device=""/>
 <part name="SUPPLY14" library="supply2" deviceset="GND" device=""/>
-<part name="RXON" library="adafruit" deviceset="R-US_" device="0204/7" value="220"/>
+<part name="RXON" library="adafruit" deviceset="R-US_" device="0204/7" value="10K"/>
 <part name="XON" library="adafruit" deviceset="LED" device="3MM"/>
 <part name="P+18" library="supply1" deviceset="+5V" device=""/>
