File: Temperature.brd (EAGLE design)
At the start: 21.6 x 26.3 mm, 3 parts, among them X1 CON

Commit message: 29/10/2013
Fixed:
-Naming in PIN
-PIR & Light Sensor PCB
Routing:
- net SIG: track 17.9 -> 25.5 mm
- net +5V: track 16.8 -> 18.6 mm
Other:
- board text added: "5v"
Changed lines of the file:
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@@
 <hole x="2.54" y="22.86" drill="3.2"/>
 <hole x="2.54" y="3.81" drill="3.2"/>
+<text x="13.97" y="3.81" size="1.016" layer="1">5v</text>
+<text x="11.43" y="22.86" size="1.016" layer="1">5v</text>
 </plain>
 <attributes>
@@
 </class>
 </classes>
-<designrules name="default">
-<description language="de">&lt;b&gt;EAGLE Design Rules&lt;/b&gt;
-&lt;p&gt;
-Die Standard-Design-Rules sind so gewählt, dass sie für
-die meisten Anwendungen passen. Sollte ihre Platine
-besondere Anforderungen haben, treffen Sie die erforderlichen
-Einstellungen hier und speichern die Design Rules unter
-einem neuen Namen ab.</description>
-<description language="en">&lt;b&gt;EAGLE Design Rules&lt;/b&gt;
+<designrules name="CUSTOM">
+<description language="id">&lt;b&gt;EAGLE Design Rules&lt;/b&gt;
 &lt;p&gt;
 The default Design Rules have been set to cover
@@
 <param name="mtCopper" value="0.035mm 0.035mm 0.035mm 0.035mm 0.035mm 0.035mm 0.035mm 0.035mm 0.035mm 0.035mm 0.035mm 0.035mm 0.035mm 0.035mm 0.035mm 0.035mm"/>
 <param name="mtIsolate" value="1.5mm 0.15mm 0.2mm 0.15mm 0.2mm 0.15mm 0.2mm 0.15mm 0.2mm 0.15mm 0.2mm 0.15mm 0.2mm 0.15mm 0.2mm"/>
-<param name="mdWireWire" value="8mil"/>
-<param name="mdWirePad" value="8mil"/>
-<param name="mdWireVia" value="8mil"/>
-<param name="mdPadPad" value="8mil"/>
-<param name="mdPadVia" value="8mil"/>
+<param name="mdWireWire" value="12mil"/>
+<param name="mdWirePad" value="12mil"/>
+<param name="mdWireVia" value="12mil"/>
+<param name="mdPadPad" value="12mil"/>
+<param name="mdPadVia" value="12mil"/>
 <param name="mdViaVia" value="8mil"/>
 <param name="mdSmdPad" value="8mil"/>
@@
 <param name="mdViaViaSameLayer" value="8mil"/>
 <param name="mnLayersViaInSmd" value="2"/>
-<param name="mdCopperDimension" value="40mil"/>
-<param name="mdDrill" value="8mil"/>
+<param name="mdCopperDimension" value="12mil"/>
+<param name="mdDrill" value="12mil"/>
 <param name="mdSmdStop" value="0mil"/>
-<param name="msWidth" value="10mil"/>
-<param name="msDrill" value="24mil"/>
+<param name="msWidth" value="12mil"/>
+<param name="msDrill" value="20mil"/>
 <param name="msMicroVia" value="9.99mm"/>
 <param name="msBlindViaRatio" value="0.5"/>
@@
 <param name="rvMicroViaOuter" value="0.25"/>
 <param name="rvMicroViaInner" value="0.25"/>
-<param name="rlMinPadTop" value="10mil"/>
+<param name="rlMinPadTop" value="12mil"/>
 <param name="rlMaxPadTop" value="20mil"/>
-<param name="rlMinPadInner" value="10mil"/>
+<param name="rlMinPadInner" value="12mil"/>
 <param name="rlMaxPadInner" value="20mil"/>
-<param name="rlMinPadBottom" value="10mil"/>
+<param name="rlMinPadBottom" value="12mil"/>
 <param name="rlMaxPadBottom" value="20mil"/>
-<param name="rlMinViaOuter" value="8mil"/>
+<param name="rlMinViaOuter" value="12mil"/>
 <param name="rlMaxViaOuter" value="20mil"/>
-<param name="rlMinViaInner" value="8mil"/>
+<param name="rlMinViaInner" value="12mil"/>
 <param name="rlMaxViaInner" value="20mil"/>
 <param name="rlMinMicroViaOuter" value="4mil"/>
@@
 <param name="mlMinCreamFrame" value="0mil"/>
 <param name="mlMaxCreamFrame" value="0mil"/>
-<param name="mlViaStopLimit" value="0mil"/>
+<param name="mlViaStopLimit" value="25mil"/>
 <param name="srRoundness" value="0"/>
 <param name="srMinRoundness" value="0mil"/>
@@
 <param name="PrefDir.14" value="0"/>
 <param name="PrefDir.15" value="0"/>
-<param name="PrefDir.16" value="/"/>
+<param name="PrefDir.16" value="0"/>
 <param name="cfVia" value="8"/>
 <param name="cfNonPref" value="5"/>
@@
 <contactref element="PULLUP" pad="2"/>
 <contactref element="DHT" pad="3"/>
-<wire x1="11.43" y1="10.16" x2="11.43" y2="8.89" width="0.254" layer="16"/>
-<wire x1="15.24" y1="13.97" x2="11.43" y2="10.16" width="0.254" layer="16"/>
-<wire x1="11.43" y1="16.51" x2="8.89" y2="19.05" width="0.254" layer="1"/>
-<wire x1="11.43" y1="8.89" x2="11.43" y2="16.51" width="0.254" layer="1"/>
+<wire x1="10.16" y1="10.16" x2="11.43" y2="8.89" width="0.3048" layer="1"/>
+<wire x1="10.16" y1="17.78" x2="10.16" y2="10.16" width="0.3048" layer="1"/>
+<wire x1="8.89" y1="19.05" x2="10.16" y2="17.78" width="0.3048" layer="1"/>
+<wire x1="15.24" y1="13.97" x2="15.24" y2="11.43" width="0.4064" layer="1"/>
+<wire x1="15.24" y1="11.43" x2="16.51" y2="10.16" width="0.4064" layer="1"/>
+<wire x1="16.51" y1="10.16" x2="16.51" y2="7.62" width="0.4064" layer="1"/>
+<wire x1="16.51" y1="7.62" x2="15.24" y2="6.35" width="0.4064" layer="1"/>
+<wire x1="15.24" y1="6.35" x2="12.7" y2="6.35" width="0.4064" layer="1"/>
+<wire x1="12.7" y1="6.35" x2="11.43" y2="7.62" width="0.4064" layer="1"/>
+<wire x1="11.43" y1="7.62" x2="11.43" y2="8.89" width="0.4064" layer="1"/>
 </signal>
 <signal name="GND">
 <contactref element="X1" pad="1"/>
 <contactref element="DHT" pad="1"/>
-<wire x1="6.35" y1="19.05" x2="6.35" y2="8.89" width="0.254" layer="1"/>
+<wire x1="6.35" y1="19.05" x2="6.35" y2="8.89" width="0.3048" layer="1"/>
 </signal>
 <signal name="+5V">
@@
 <contactref element="DHT" pad="4"/>
 <contactref element="PULLUP" pad="1"/>
-<wire x1="12.7" y1="8.89" x2="13.97" y2="8.89" width="0.254" layer="1"/>
-<wire x1="12.7" y1="17.78" x2="12.7" y2="8.89" width="0.254" layer="1"/>
-<wire x1="11.43" y1="19.05" x2="12.7" y2="17.78" width="0.254" layer="1"/>
-<wire x1="13.97" y1="21.59" x2="15.24" y2="21.59" width="0.254" layer="16"/>
-<wire x1="11.43" y1="19.05" x2="13.97" y2="21.59" width="0.254" layer="16"/>
+<wire x1="12.7" y1="10.16" x2="13.97" y2="8.89" width="0.3048" layer="1"/>
+<wire x1="12.7" y1="17.78" x2="12.7" y2="15.24" width="0.3048" layer="1"/>
+<wire x1="12.7" y1="15.24" x2="12.7" y2="10.16" width="0.3048" layer="1"/>
+<wire x1="11.43" y1="19.05" x2="12.7" y2="17.78" width="0.3048" layer="1"/>
+<wire x1="15.24" y1="21.59" x2="15.24" y2="17.78" width="0.4064" layer="1"/>
+<wire x1="15.24" y1="17.78" x2="12.7" y2="15.24" width="0.4064" layer="1"/>
 </signal>
 </signals>
