File: Control.brd (EAGLE design)
At the start: 106.7 x 83.5 mm, 44 parts, among them IC2 7805T, IC3 LP2950Z, Q2 16MHZ, X1 BUT4, X10 DIG2, X11 DIG3, X12 DIG4, X2 BUT3, X3 AL1, X4 BUT2, X5 BUT1, X6 AL2, X7 AL3, X8 AL4, X9 DIG1

Commit message: 28/10/13
Fixed:
-Relay PCB
-half Control PCB

unfixed:
-Control PCB GND separation
Parts:
- removed PDM, PDM1, PDS, PDS1: 10k, adafruit:0204/7
- added PDBUT1, PDBUT2, PDBUT3, PDBUT4: 10k, adafruit:0204/7
- moved PSCL 117.1 mm to (57.1, 10.2), turned to 270 degrees
- moved PSDA 112.5 mm to (54.6, 10.2), turned to 270 degrees
- moved X9 110.7 mm to (11.4, 50.8), turned to 270 degrees
- moved X11 104.3 mm to (11.4, 33.0), turned to 270 degrees
- moved JP2 102.9 mm to (49.5, 8.89)
- moved X10 101.6 mm to (11.4, 41.9), turned to 270 degrees
- moved X12 95.3 mm to (11.4, 24.1), turned to 270 degrees
- moved JP1 89.2 mm to (11.4, 16.5)
- moved X8 65.2 mm to (40.6, 6.35)
- moved X3 60.4 mm to (14.0, 6.35)
- moved X1 59.5 mm to (20.3, 50.8)
- moved X2 59.5 mm to (26.7, 50.8)
- moved X7 50.8 mm to (31.8, 6.35)
- moved JP4 36.6 mm to (55.9, 27.9), turned to 180 degrees
- moved X6 36.4 mm to (22.9, 6.35)
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Connections:
- net BUT1: now also PDBUT1.2; no longer PDS.2
- net BUT2: now also PDBUT2.2; no longer PDM.2
- net BUT3: now also PDBUT3.2; no longer PDS1.2
- net BUT4: now also PDBUT4.2; no longer PDM1.2
- net GND: now also PDBUT1.1, PDBUT2.1, PDBUT3.1, PDBUT4.1; no longer PDM.1, PDM1.1, PDS.1, PDS1.1
Routing:
- net GND: track 372.4 -> 0.00 mm
- net +5V: track 256.8 -> 0.00 mm
- net VCC: track 171.6 -> 0.00 mm
- net +3V3: track 107.4 -> 0.00 mm
- net DIG1: track 0.00 -> 66.1 mm
- net N$7: track 56.2 -> 0.00 mm
- net AGND: track 62.8 -> 12.5 mm
- net BUT1: track 31.9 -> 0.00 mm
- net TX: track 30.1 -> 0.00 mm
- net N$1: track 26.8 -> 0.00 mm
- net AL2: track 0.00 -> 23.7 mm
- net RX: track 22.1 -> 0.00 mm
- net BUT4: track 20.6 -> 0.00 mm
- net N$29: track 20.4 -> 0.00 mm
- net AL1: track 11.5 -> 30.0 mm
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- added copper zone on layer 16, net +5V
- added copper zone on layer 1, net GND
- removed copper zone on layer 16, net AGND
- removed copper zone on layer 16, net GND
Other:
- board size 106.7 x 83.5 mm -> 85.1 x 59.4 mm

Commit message: 28/10/13 - 2
Fixed:
-Relay & Control PCB

Unfixed:
-IR PCB
-Temperature PCB
Parts:
- moved REF 43.5 mm to (17.8, 6.35)
- moved JP2 13.3 mm to (62.2, 5.08), turned to 90 degrees
- moved X6 10.2 mm to (33.0, 6.35)
- moved X3 10.2 mm to (24.1, 6.35)
- moved X7 10.2 mm to (41.9, 6.35)
- moved X8 10.2 mm to (50.8, 6.35)
- moved U$1 8.98 mm to (83.8, 11.4)
- moved IC3 7.62 mm to (74.9, 38.1)
- moved AGND 5.24 mm to (55.9, 5.08)
- moved REG3O 5.08 mm to (74.9, 31.8), turned to 0 degrees
- moved PSCL 3.81 mm to (57.1, 14.0), turned to 0 degrees
- moved Q2 3.81 mm to (31.8, 31.8)
- moved PSDA 2.84 mm to (57.1, 11.4), turned to 0 degrees
- moved C3 2.54 mm to (29.2, 35.6)
- moved C4 2.54 mm to (35.6, 35.6)
Connections:
- net +5V: now also JP2.1
- net VCC: no longer JP2.1
Routing:
- net VCC: track 0.00 -> 129.5 mm
- net +5V: track 0.00 -> 95.0 mm
- net DIG2: track 0.00 -> 45.5 mm
- net BUT2: track 0.00 -> 39.2 mm
- net TX: track 0.00 -> 38.4 mm
- net BUT4: track 0.00 -> 38.2 mm
- net BUT3: track 0.00 -> 36.0 mm
- net BUT1: track 0.00 -> 33.9 mm
- net +3V3: track 0.00 -> 30.8 mm
- net RX: track 0.00 -> 29.3 mm
- net REL4: track 0.00 -> 23.7 mm
- net AGND: track 12.5 -> 34.7 mm
- net N$2: track 0.00 -> 21.6 mm
- net DIG3: track 0.00 -> 21.2 mm
- net N$1: track 0.00 -> 20.4 mm
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- added copper zone on layer 16, net AGND

Commit message: 29/10/2013
Fixed:
-Naming in PIN
-PIR & Light Sensor PCB
Other:
- board text added: "REL1"
- board text added: "VCC"
Changed lines of the file:
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@@
 <hole x="81.28" y="55.88" drill="3.2"/>
 <hole x="3.81" y="55.88" drill="3.2"/>
+<text x="3.81" y="13.97" size="0.8128" layer="1">VCC</text>
+<text x="11.43" y="10.16" size="0.8128" layer="1" rot="R90">REL1</text>
 </plain>
 <attributes>

Commit message: 11/10/3
FIXED:
-connector
-refine route
Parts:
- removed JP1: RELAY, pinhead:2X03
- removed JP2: I2C, pinhead:2X02
- added I2C: I2C, con-molex:22-23-2041
- added RELAY: RELAY, con-molex:22-23-2061
- moved AGND 1.27 mm to (55.9, 6.35)
Connections:
- net +5V: now also I2C.4; no longer JP2.1
- net GND: now also I2C.1, RELAY.1; no longer JP1.2, JP2.3
- net REL1: now also RELAY.5; no longer JP1.3
- net REL2: now also RELAY.4; no longer JP1.4
- net REL3: now also RELAY.3; no longer JP1.5
- net REL4: now also RELAY.2; no longer JP1.6
- net SCL: now also I2C.2; no longer JP2.4
- net SDA: now also I2C.3; no longer JP2.2
- net VCC: now also RELAY.6; no longer JP1.1
Routing:
- net GND: track 0.00 -> 25.2 mm
- net SCL: track 14.3 -> 30.8 mm
- net REL2: track 14.3 -> 25.0 mm
- net VCC: track 129.5 -> 137.2 mm
- net REL4: track 23.7 -> 21.2 mm
- net N$2: track 21.6 -> 20.1 mm
- net REL3: track 14.6 -> 16.1 mm
- net SDA: track 17.8 -> 19.1 mm
- net +5V: track 95.0 -> 96.0 mm
- net AGND: track 34.7 -> 34.2 mm
Other:
- board text removed: "REL1"
- board text removed: "VCC"

Commit message: 13/11/13
Fixed:
-Resistor Value
Parts:
- RXASC, RXON: value 220 -> 10K
Changed lines of the file:
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@@
 <element name="U$1" library="adafruit" package="PJ-102A" value="2.1MMJACKTHM" x="83.82" y="11.43" rot="R270"/>
 <element name="U$4" library="SparkFun-RF" package="XBEE-1" value="XBEE-1B1" x="71.12" y="43.18" rot="R90"/>
-<element name="RXASC" library="adafruit" package="0204/7" value="220" x="66.04" y="48.26"/>
+<element name="RXASC" library="adafruit" package="0204/7" value="10K" x="66.04" y="48.26"/>
 <element name="XASC" library="adafruit" package="LED3MM" value="" x="74.93" y="48.26"/>
 <element name="RSSI1" library="adafruit" package="1X01" value="" x="74.93" y="43.18"/>
 <element name="XDIV1" library="adafruit" package="0204/7" value="10K" x="50.8" y="35.56"/>
 <element name="XDIV2" library="adafruit" package="0204/7" value="15K" x="50.8" y="38.1"/>
-<element name="RXON" library="adafruit" package="0204/7" value="220" x="66.04" y="50.8"/>
+<element name="RXON" library="adafruit" package="0204/7" value="10K" x="66.04" y="50.8"/>
 <element name="XON" library="adafruit" package="LED3MM" value="" x="74.93" y="53.34"/>
 <element name="AGND" library="adafruit" package="1X01" value="AGND" x="55.88" y="6.35"/>
