File: Relay30.brd (EAGLE design)
At the start: 119.4 x 55.5 mm, 33 parts

Commit message: 29/10/2013
Fixed:
-Naming in PIN
-PIR & Light Sensor PCB
Other:
- board text added: "GND"
- board text added: "REL3"
- board text added: "REL4"
Changed lines of the file:
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@@
 <setting verticaltext="up"/>
 </settings>
-<grid distance="0.05" unitdist="inch" unit="mm" style="lines" multiple="1" display="yes" altdistance="0.025" altunitdist="inch" altunit="inch"/>
+<grid distance="0.7" unitdist="mm" unit="mm" style="lines" multiple="1" display="yes" altdistance="0.025" altunitdist="inch" altunit="inch"/>
 <layers>
 <layer number="1" name="Top" color="4" fill="1" visible="yes" active="yes"/>
@@
 <hole x="115.57" y="52.07" drill="3.2"/>
 <hole x="115.57" y="3.81" drill="3.2"/>
+<text x="63" y="51.8" size="0.8128" layer="1">GND</text>
+<text x="63" y="49" size="0.8128" layer="1">REL3</text>
+<text x="63" y="46.2" size="0.8128" layer="1">REL4</text>
 </plain>
 <attributes>

Commit message: 11/10/3
FIXED:
-connector
-refine route
Parts:
- removed JP1: RELAY, pinhead:2X03
- added X1: (no value), con-molex:22-23-2061
- moved RELAY1 1.05 mm to (17.1, 25.8)
- moved RELAY4 0.79 mm to (103.6, 26.1)
- moved RELAY3 0.61 mm to (74.7, 26.1)
- moved RELAY2 0.58 mm to (45.8, 26.1)
- moved FLY2 0.30 mm to (49.5, 48.0)
- moved FLY3 0.30 mm to (81.3, 48.0)
Connections:
- net GND: now also X1.1; no longer JP1.2
- net REL1: now also X1.5; no longer JP1.3
- net REL2: now also X1.4; no longer JP1.5
- net REL3: now also X1.3; no longer JP1.4
- net REL4: now also X1.2; no longer JP1.6
- net VCC: now also X1.6; no longer JP1.1
Routing:
- net VCC: track 289.7 -> 274.2 mm
- net REL1: track 57.9 -> 51.1 mm
- net N$2: track 55.8 -> 58.4 mm
- net N$7: track 40.8 -> 42.6 mm
- net REL4: track 35.4 -> 34.2 mm
- net GND: track 121.3 -> 120.2 mm
- net REL2: track 28.8 -> 27.7 mm
- net N$17: track 41.0 -> 40.1 mm
- net N$11: track 10.8 -> 11.6 mm
- net N$1: track 16.2 -> 15.4 mm
- net N$12: track 43.7 -> 44.3 mm
Other:
- board text removed: "GND"
- board text removed: "REL3"
- board text removed: "REL4"

Commit message: 13/11/13
Fixed:
-Resistor Value
Parts:
- RRELED1, RRELED2, RRELED3, RRELED4: value 470 -> 10K
Changed lines of the file:
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@@
 <element name="TREL1" library="transistor" package="TO92" value="2N3904" x="25.4" y="49.53"/>
 <element name="RELIND1" library="adafruit" package="LED3MM" value="" x="25.4" y="45.72" rot="R90"/>
-<element name="RRELED1" library="adafruit" package="0204/7" value="470" x="17.78" y="45.72"/>
+<element name="RRELED1" library="adafruit" package="0204/7" value="10K" x="17.78" y="45.72"/>
 <element name="REL1" library="SparkFun-Connectors" package="SCREWTERMINAL-5MM-2" value="TERM" x="13.97" y="5.08"/>
 <element name="FLY2" library="adafruit" package="DO-1N4148" value="" x="49.53" y="47.96" rot="R90"/>
@@
 <element name="TREL2" library="transistor" package="TO92" value="2N3904" x="44.45" y="49.53"/>
 <element name="RELIND2" library="adafruit" package="LED3MM" value="" x="44.45" y="45.72" rot="R90"/>
-<element name="RRELED2" library="adafruit" package="0204/7" value="470" x="35.56" y="45.72"/>
+<element name="RRELED2" library="adafruit" package="0204/7" value="10K" x="35.56" y="45.72"/>
 <element name="REL2" library="SparkFun-Connectors" package="SCREWTERMINAL-5MM-2" value="TERM" x="41.91" y="5.08"/>
 <element name="FLY3" library="adafruit" package="DO-1N4148" value="" x="81.28" y="47.96" rot="R90"/>
@@
 <element name="TREL3" library="transistor" package="TO92" value="2N3904" x="86.36" y="49.53"/>
 <element name="RELIND3" library="adafruit" package="LED3MM" value="" x="86.36" y="45.72" rot="R90"/>
-<element name="RRELED3" library="adafruit" package="0204/7" value="470" x="74.93" y="45.72"/>
+<element name="RRELED3" library="adafruit" package="0204/7" value="10K" x="74.93" y="45.72"/>
 <element name="REL3" library="SparkFun-Connectors" package="SCREWTERMINAL-5MM-2" value="TERM" x="71.12" y="5.08"/>
 <element name="FLY4" library="adafruit" package="DO-1N4148" value="" x="101.6" y="48.26" rot="R90"/>
@@
 <element name="TREL4" library="transistor" package="TO92" value="2N3904" x="106.68" y="49.53"/>
 <element name="RELIND4" library="adafruit" package="LED3MM" value="" x="106.68" y="45.72" rot="R90"/>
-<element name="RRELED4" library="adafruit" package="0204/7" value="470" x="95.25" y="45.72"/>
+<element name="RRELED4" library="adafruit" package="0204/7" value="10K" x="95.25" y="45.72"/>
 <element name="REL4" library="SparkFun-Connectors" package="SCREWTERMINAL-5MM-2" value="TERM" x="100.33" y="5.08"/>
 <element name="X1" library="con-molex" package="22-23-2061" value="" x="60.2" y="48.3" rot="R180">
