File: Relay30.sch (EAGLE design)
At the start: 33 parts

Commit message: 11/10/3
FIXED:
-connector
-refine route
Parts:
- removed JP1: RELAY, pinhead:PINHD-2X3
- added X1: (no value), con-molex:22-23-2061
Connections:
- net GND: now also X1-1.S; no longer JP1.2
- net REL1: now also X1-5.S; no longer JP1.3
- net REL2: now also X1-4.S; no longer JP1.5
- net REL3: now also X1-3.S; no longer JP1.4
- net REL4: now also X1-2.S; no longer JP1.6
- net VCC: now also X1-6.S; no longer JP1.1

Commit message: 13/11/13
Fixed:
-Resistor Value
Parts:
- RRELED1, RRELED2, RRELED3, RRELED4: value 470 -> 10K
Changed lines of the file:
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@@
 <part name="SUPPLY2" library="supply2" deviceset="GND" device=""/>
 <part name="RELIND1" library="adafruit" deviceset="LED" device="3MM"/>
-<part name="RRELED1" library="adafruit" deviceset="R-US_" device="0204/7" value="470"/>
+<part name="RRELED1" library="adafruit" deviceset="R-US_" device="0204/7" value="10K"/>
 <part name="SUPPLY6" library="supply2" deviceset="GND" device=""/>
 <part name="REL1" library="SparkFun-Connectors" deviceset="M02" device="5MM" value="TERM"/>
@@
 <part name="SUPPLY4" library="supply2" deviceset="GND" device=""/>
 <part name="RELIND2" library="adafruit" deviceset="LED" device="3MM"/>
-<part name="RRELED2" library="adafruit" deviceset="R-US_" device="0204/7" value="470"/>
+<part name="RRELED2" library="adafruit" deviceset="R-US_" device="0204/7" value="10K"/>
 <part name="REL2" library="SparkFun-Connectors" deviceset="M02" device="5MM" value="TERM"/>
 <part name="FLY3" library="adafruit" deviceset="DIODE" device="DO-1N4148"/>
@@
 <part name="SUPPLY7" library="supply2" deviceset="GND" device=""/>
 <part name="RELIND3" library="adafruit" deviceset="LED" device="3MM"/>
-<part name="RRELED3" library="adafruit" deviceset="R-US_" device="0204/7" value="470"/>
+<part name="RRELED3" library="adafruit" deviceset="R-US_" device="0204/7" value="10K"/>
 <part name="REL3" library="SparkFun-Connectors" deviceset="M02" device="5MM" value="TERM"/>
 <part name="FLY4" library="adafruit" deviceset="DIODE" device="DO-1N4148"/>
@@
 <part name="SUPPLY9" library="supply2" deviceset="GND" device=""/>
 <part name="RELIND4" library="adafruit" deviceset="LED" device="3MM"/>
-<part name="RRELED4" library="adafruit" deviceset="R-US_" device="0204/7" value="470"/>
+<part name="RRELED4" library="adafruit" deviceset="R-US_" device="0204/7" value="10K"/>
 <part name="REL4" library="SparkFun-Connectors" deviceset="M02" device="5MM" value="TERM"/>
 <part name="SUPPLY10" library="supply2" deviceset="VCC" device=""/>
